File: 5. Semester/Electroacoustics/Labs/Lab A/KiCad/Part2a_Silencer_PressureSource/Part2a_Silencer_PressureSource.kicad_sch (KiCad schematic)
At the start: 16 parts

Commit message: Lab A report: correct the part 2 silencer numbers and figures
Rerun part 2 with an unloaded volume-velocity source (1 T instead of the
100 Meg leak) and 2000 points per decade: three peaks of +38.6/+40.9/+41.1 dB
at 47/176/191 Hz, 2a peaks -98.9/-112.3/-141.6 dB, tables 2a-2e, the 10 m SPL
and the conclusions updated; the report now records the leak-resistor trap.
Other:
- note added: ".ac dec 2000 10 1000"
- note removed: ".ac dec 200 10 1000"
Changed lines of the file:
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@@
 		)
 	)
-	(text ".ac dec 200 10 1000"
+	(text ".ac dec 2000 10 1000"
 		(at 190.5 17.78 0)
 		(effects
@@
 		(instances
 			(project "Part2a_Silencer_PressureSource"
-				(path "/44785935-fb4a-4bdf-8b33-a4d8f2d9b238"
+				(path "/5845d250-878a-4d29-bb06-e0d60c4645a2"
 					(reference "V1")
 					(unit 1)
@@
 		(instances
 			(project "Part2a_Silencer_PressureSource"
-				(path "/44785935-fb4a-4bdf-8b33-a4d8f2d9b238"
+				(path "/5845d250-878a-4d29-bb06-e0d60c4645a2"
 					(reference "Vs1")
 					(unit 1)
@@
 		(instances
 			(project "Part2a_Silencer_PressureSource"
-				(path "/44785935-fb4a-4bdf-8b33-a4d8f2d9b238"
+				(path "/5845d250-878a-4d29-bb06-e0d60c4645a2"
 					(reference "R1")
 					(unit 1)
@@
 		(instances
 			(project "Part2a_Silencer_PressureSource"
-				(path "/44785935-fb4a-4bdf-8b33-a4d8f2d9b238"
+				(path "/5845d250-878a-4d29-bb06-e0d60c4645a2"
 					(reference "L1")
 					(unit 1)
@@
 		(instances
 			(project "Part2a_Silencer_PressureSource"
-				(path "/44785935-fb4a-4bdf-8b33-a4d8f2d9b238"
+				(path "/5845d250-878a-4d29-bb06-e0d60c4645a2"
 					(reference "C2")
 					(unit 1)
@@
 		(instances
 			(project "Part2a_Silencer_PressureSource"
-				(path "/44785935-fb4a-4bdf-8b33-a4d8f2d9b238"
+				(path "/5845d250-878a-4d29-bb06-e0d60c4645a2"
 					(reference "Vs3")
 					(unit 1)
@@
 		(instances
 			(project "Part2a_Silencer_PressureSource"
-				(path "/44785935-fb4a-4bdf-8b33-a4d8f2d9b238"
+				(path "/5845d250-878a-4d29-bb06-e0d60c4645a2"
 					(reference "R3")
 					(unit 1)
@@
 		(instances
 			(project "Part2a_Silencer_PressureSource"
-				(path "/44785935-fb4a-4bdf-8b33-a4d8f2d9b238"
+				(path "/5845d250-878a-4d29-bb06-e0d60c4645a2"
 					(reference "L3")
 					(unit 1)
@@
 		(instances
 			(project "Part2a_Silencer_PressureSource"
-				(path "/44785935-fb4a-4bdf-8b33-a4d8f2d9b238"
+				(path "/5845d250-878a-4d29-bb06-e0d60c4645a2"
 					(reference "C4")
 					(unit 1)
@@
 		(instances
 			(project "Part2a_Silencer_PressureSource"
-				(path "/44785935-fb4a-4bdf-8b33-a4d8f2d9b238"
+				(path "/5845d250-878a-4d29-bb06-e0d60c4645a2"
 					(reference "Vs5")
 					(unit 1)
@@
 		(instances
 			(project "Part2a_Silencer_PressureSource"
-				(path "/44785935-fb4a-4bdf-8b33-a4d8f2d9b238"
+				(path "/5845d250-878a-4d29-bb06-e0d60c4645a2"
 					(reference "R5")
 					(unit 1)
@@
 		(instances
 			(project "Part2a_Silencer_PressureSource"
-				(path "/44785935-fb4a-4bdf-8b33-a4d8f2d9b238"
+				(path "/5845d250-878a-4d29-bb06-e0d60c4645a2"
 					(reference "L5")
 					(unit 1)
@@
 		(instances
 			(project "Part2a_Silencer_PressureSource"
-				(path "/44785935-fb4a-4bdf-8b33-a4d8f2d9b238"
+				(path "/5845d250-878a-4d29-bb06-e0d60c4645a2"
 					(reference "C6")
 					(unit 1)
@@
 		(instances
 			(project "Part2a_Silencer_PressureSource"
-				(path "/44785935-fb4a-4bdf-8b33-a4d8f2d9b238"
+				(path "/5845d250-878a-4d29-bb06-e0d60c4645a2"
 					(reference "Vs7")
 					(unit 1)
@@
 		(instances
 			(project "Part2a_Silencer_PressureSource"
-				(path "/44785935-fb4a-4bdf-8b33-a4d8f2d9b238"
+				(path "/5845d250-878a-4d29-bb06-e0d60c4645a2"
 					(reference "R7")
 					(unit 1)
@@
 		(instances
 			(project "Part2a_Silencer_PressureSource"
-				(path "/44785935-fb4a-4bdf-8b33-a4d8f2d9b238"
+				(path "/5845d250-878a-4d29-bb06-e0d60c4645a2"
 					(reference "L7")
 					(unit 1)
@@
 		(instances
 			(project "Part2a_Silencer_PressureSource"
-				(path "/44785935-fb4a-4bdf-8b33-a4d8f2d9b238"
+				(path "/5845d250-878a-4d29-bb06-e0d60c4645a2"
 					(reference "#PWR001")
 					(unit 1)
@@
 		(instances
 			(project "Part2a_Silencer_PressureSource"
-				(path "/44785935-fb4a-4bdf-8b33-a4d8f2d9b238"
+				(path "/5845d250-878a-4d29-bb06-e0d60c4645a2"
 					(reference "#PWR002")
 					(unit 1)
